File: ATmega328P/Schematics/ATmega328P_CustomBd_LCD_RTCDS1307_DHT11.sch (EAGLE design)
At the start: 18 parts, among them IC1 ATMEGA328-20P, IC2 DS1307, Q1 32.768 Khz, X1 HD44780LCD-1602

Commit message: Vo w/2K2 and GND not to Vcc
Vo(Contrast of LCD) connection to Vcc has been modified to GND.
Connections:
- net GND: now also R5.1
- net N$10: no longer C1.2
- net VCC: no longer R5.1
Other:
- note added: "Source code C:\Users\insoo\Documents\GitHub\ATmelStudio\ATmega328P\Schematics (on github.com Desktop)"
- note removed: "Source code C:\Users\insoo\Box Sync\BoxElec\DIY Electronics\Arduino\AVR C\Win_Atmel Studio_Codes\7.0\ATmega328P\LCD\LCD_RTC_DS1307_DHT11 (on Box.com)"
- moved on the sheet: C1, R5
Changed lines of the file:
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@@
 <part name="GND3" library="supply1" deviceset="GND" device=""/>
 <part name="FRAME1" library="frames" deviceset="LETTER_L" device=""/>
-<part name="P+4" library="supply1" deviceset="VCC" device=""/>
 <part name="IC2" library="adafruit" library_urn="urn:adsk.eagle:library:420" deviceset="DS1307" device=""/>
 <part name="GND5" library="supply1" deviceset="GND" device=""/>
@@
 <part name="G1" library="battery" library_urn="urn:adsk.eagle:library:109" deviceset="CR2032H" device=""/>
 <part name="X1" library="adafruit" library_urn="urn:adsk.eagle:library:420" deviceset="HD44780LCD" device="-1602"/>
+<part name="GND4" library="supply1" deviceset="GND" device=""/>
 </parts>
 <sheets>
@@
 <text x="-30.48" y="147.32" size="1.778" layer="91">#define DHT_VCC_bit PORTB2</text>
 <text x="-10.16" y="248.92" size="1.778" layer="91">#define DS1307_VCC_bit PORTB7</text>
-<text x="-60.96" y="101.6" size="1.778" layer="91">Source code C:\Users\insoo\Box Sync\BoxElec\DIY Electronics\Arduino\AVR C\Win_Atmel Studio_Codes\7.0\ATmega328P\LCD\LCD_RTC_DS1307_DHT11  (on Box.com)</text>
+<text x="-60.96" y="101.6" size="1.778" layer="91">Source code C:\Users\insoo\Documents\GitHub\ATmelStudio\ATmega328P\Schematics  (on github.com Desktop)</text>
 </plain>
 <instances>
@@
 <instance part="R3" gate="G$1" x="-15.24" y="142.24" rot="R90"/>
 <instance part="R4" gate="G$1" x="20.32" y="167.64"/>
-<instance part="R5" gate="G$1" x="0" y="218.44" rot="R270"/>
+<instance part="R5" gate="G$1" x="5.08" y="215.9" rot="R270"/>
 <instance part="R6" gate="G$1" x="-45.72" y="231.14"/>
-<instance part="C1" gate="G$1" x="27.94" y="180.34"/>
+<instance part="C1" gate="G$1" x="30.48" y="187.96"/>
 <instance part="SV1" gate="G$1" x="114.3" y="167.64" rot="MR0"/>
 <instance part="P+1" gate="VCC" x="99.06" y="134.62"/>
@@
 <instance part="SV2" gate="G$1" x="134.62" y="167.64" rot="MR0"/>
 <instance part="JP3" gate="A" x="-2.54" y="185.42" rot="MR0"/>
-<instance part="P+2" gate="VCC" x="25.4" y="208.28"/>
+<instance part="P+2" gate="VCC" x="25.4" y="177.8"/>
 <instance part="U$1" gate="G$1" x="-15.24" y="121.92" rot="R180"/>
 <instance part="GND3" gate="1" x="-27.94" y="132.08"/>
 <instance part="FRAME1" gate="G$1" x="-60.96" y="73.66"/>
 <instance part="FRAME1" gate="G$2" x="86.36" y="73.66"/>
-<instance part="P+4" gate="VCC" x="0" y="226.06"/>
 <instance part="IC2" gate="G$1" x="-22.86" y="228.6"/>
 <instance part="GND5" gate="1" x="-22.86" y="210.82"/>
@@
 <instance part="G1" gate="1" x="-12.7" y="213.36"/>
 <instance part="X1" gate="G$1" x="-27.94" y="180.34" rot="R270"/>
+<instance part="GND4" gate="1" x="-2.54" y="218.44"/>
 </instances>
 <busses>
@@
 <junction x="22.86" y="193.04"/>
 <pinref part="C1" gate="G$1" pin="1"/>
-<wire x1="27.94" y1="182.88" x2="27.94" y2="190.5" width="0.1524" layer="91"/>
 <pinref part="IC1" gate="G$1" pin="GND"/>
 <wire x1="27.94" y1="190.5" x2="30.48" y2="190.5" width="0.1524" layer="91"/>
@@
 <pinref part="G1" gate="1" pin="-"/>
 <wire x1="-17.78" y1="213.36" x2="-22.86" y2="213.36" width="0.1524" layer="91"/>
+</segment>
+<segment>
+<pinref part="GND4" gate="1" pin="GND"/>
+<pinref part="R5" gate="G$1" pin="1"/>
+<wire x1="-2.54" y1="220.98" x2="5.08" y2="220.98" width="0.1524" layer="91"/>
 </segment>
 </net>
@@
 </segment>
 <segment>
-<pinref part="R5" gate="G$1" pin="1"/>
-<pinref part="P+4" gate="VCC" pin="VCC"/>
-</segment>
-<segment>
 <pinref part="R7" gate="G$1" pin="1"/>
 <pinref part="P+3" gate="VCC" pin="VCC"/>
@@
 <pinref part="P+2" gate="VCC" pin="VCC"/>
 <pinref part="R4" gate="G$1" pin="2"/>
-<wire x1="25.4" y1="205.74" x2="25.4" y2="172.72" width="0.1524" layer="91"/>
+<wire x1="25.4" y1="175.26" x2="25.4" y2="172.72" width="0.1524" layer="91"/>
 <pinref part="IC1" gate="G$1" pin="VCC"/>
 <wire x1="25.4" y1="172.72" x2="25.4" y2="167.64" width="0.1524" layer="91"/>
 <wire x1="30.48" y1="185.42" x2="30.48" y2="172.72" width="0.1524" layer="91"/>
-<pinref part="C1" gate="G$1" pin="2"/>
-<wire x1="30.48" y1="172.72" x2="27.94" y2="172.72" width="0.1524" layer="91"/>
-<wire x1="27.94" y1="172.72" x2="27.94" y2="175.26" width="0.1524" layer="91"/>
-<wire x1="27.94" y1="172.72" x2="25.4" y2="172.72" width="0.1524" layer="91"/>
+<wire x1="30.48" y1="172.72" x2="25.4" y2="172.72" width="0.1524" layer="91"/>
 </segment>
 </net>
@@
 <segment>
 <pinref part="R5" gate="G$1" pin="2"/>
-<wire x1="0" y1="213.36" x2="5.08" y2="213.36" width="0.1524" layer="91"/>
-<wire x1="5.08" y1="213.36" x2="5.08" y2="198.12" width="0.1524" layer="91"/>
+<wire x1="5.08" y1="210.82" x2="5.08" y2="213.36" width="0.1524" layer="91"/>
+<wire x1="5.08" y1="210.82" x2="5.08" y2="198.12" width="0.1524" layer="91"/>
 <pinref part="JP3" gate="A" pin="3"/>
 <wire x1="5.08" y1="198.12" x2="0" y2="198.12" width="0.1524" layer="91"/>
